File: Simplified RGB Controller.kicad_pcb (KiCad board)
At the start: 2 copper layers, 52.1 x 85.1 mm, 16 parts, among them IC1 SN74HCT245DBR, J1 RGB_3_pin, J2 RGB_3_pin, J3 RGB_3_pin, J4 RGB_3_pin, J5 RGB_3_pin, J6 RGB_3_pin, J7 RGB_3_pin, J8 RGB_3_pin, J9 AMP_Mate-N-Lok_Power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

Commit message: * Incoporate feedback * The ESP32 takes 12V on VIN
Parts:
- removed D1: 1N5819HW-7-F, local:SOD3716X145N
- added 100nF: C_Small, Capacitor_SMD:C_0603_1608Metric_Pad1.08x0.95mm_HandSolder, F.Cu at (169.3, 77.5)
- J9: value AMP_Mate-N-Lok_Power -> Molex Power
- moved IC1 20.3 mm to (162.6, 82.5)
- moved J9 3.81 mm to (153.7, 68.6)
Connections:
- IC1 pad 20: +5V -> Net-(C1-Pad1)
- J9 pad 1: Net-(J9-Pad1) -> +12V
- U1 pad 15: Net-(D1-Pad1) -> +12V
Routing:
- net +12V: track 0.00 -> 63.9 mm
- net +5V: track 174.2 -> 126.8 mm
- net /B8: track 45.9 -> 67.2 mm
- net /B7: track 37.1 -> 57.8 mm
- net /A3: track 14.0 -> 34.5 mm
- net /A7: track 21.1 -> 41.4 mm
- net /A4: track 15.5 -> 35.7 mm
- net /A6: track 19.3 -> 39.5 mm
- net /A8: track 23.0 -> 43.3 mm
- net /A5: track 17.4 -> 37.6 mm
- net /B6: track 29.1 -> 48.3 mm
- net /A2: track 13.2 -> 32.0 mm
- net /A1: track 12.4 -> 30.1 mm
- net /B1: track 41.1 -> 26.5 mm
- net /B5: track 25.1 -> 38.8 mm
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Other:
- board text added: "12V"
- board text added: "5V"

Commit message: Update to match parts available at JCL.
Parts:
- removed 100nF: C_Small, Capacitor_SMD:C_0603_1608Metric_Pad1.08x0.95mm_HandSolder
- added C1: 100nF, Capacitor_SMD:C_0603_1608Metric, F.Cu at (167.1, 77.5)
- IC1: value SN74HCT245DBR -> SN74HCT245PWR
- J9: value Molex Power -> AMP_Mate-N-Lok_Power; footprint local:AMP_Mate_N_Lok -> local:TE_MATE-N-LOK_350211-1_1x04_P5.08mm_Vertical
- turned J9 to 0 degrees
Connections:
- IC1 pad 20: Net-(C1-Pad1) -> +5V
Routing:
- net Net-(C1-Pad1): track 3.50 -> 0.00 mm
- net +5V: track 126.8 -> 124.1 mm
- net GND: track 5.32 -> 6.82 mm
Other:
- board text added: "JLCJLCJLCJLC"
